File: Yaesu to CIV.brd (EAGLE design)
At the start: 24.9 x 20.9 mm, 54 parts, among them IC1 MEGA8-AI, IC2 MC78M05CDTG, Q1 16Mhz, Q2 BC849SMD, Q3 BC849SMD, Q4 BC849SMD

Commit message: Add files via upload
Parts:
- added LED1: (no value), led:CHIP-LED0603
- added R16: 470R7, rcl:R0603
- moved C3 0.32 mm to (8.57, 13.5)
Connections:
- new net C: IC1.19, LED1.A
- new net N$36: LED1.C, R16.1
- net GND: now also R16.2
Routing:
- net C: track 0.00 -> 4.37 mm, vias 0 -> 1
- net N$37: track 0.00 -> 1.49 mm
- net N$1: track 9.47 -> 9.99 mm
