File: Yaesu to CIV.brd (EAGLE design)
At the start: 24.9 x 20.9 mm, 56 parts, among them IC1 MEGA8-AI, IC2 MC78M05CDTG, Q1 16Mhz, Q2 BC849SMD, Q3 BC849SMD, Q4 BC849SMD

Commit message: Add files via upload
Connections:
- removed net C: IC1.19, LED1.A
- net N$24: now also LED1.A
Routing:
- net C: track 4.37 -> 0.00 mm, vias 1 -> 0
- net N$24: track 5.38 -> 8.32 mm, vias 0 -> 1
Changed lines of the file:
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@@
 <contactref element="X1" pad="6"/>
 <via x="3.81" y="14.605" extent="1-16" drill="0.2"/>
-<via x="7.62" y="7.14375" extent="1-16" drill="0.2"/>
+<via x="9.68375" y="8.5725" extent="1-16" drill="0.2"/>
 <contactref element="C12" pad="2"/>
 <via x="3.81" y="15.08125" extent="1-16" drill="0.2"/>
@@
 <via x="23.97125" y="0.47625" extent="1-16" drill="0.2"/>
 <via x="11.1125" y="5.55625" extent="1-16" drill="0.2"/>
-<via x="10.95375" y="7.62" extent="1-16" drill="0.2"/>
+<via x="10.795" y="7.46125" extent="1-16" drill="0.2"/>
 <via x="13.81125" y="10.63625" extent="1-16" drill="0.2"/>
 <via x="10.4775" y="11.58875" extent="1-16" drill="0.2"/>
@@
 <wire x1="6.0325" y1="10.16" x2="4.92125" y2="11.27125" width="0.1524" layer="1"/>
 <wire x1="4.92125" y1="11.27125" x2="4.92125" y2="15.08125" width="0.1524" layer="1"/>
+<contactref element="LED1" pad="A"/>
+<wire x1="6.0325" y1="10.00125" x2="5.3975" y2="9.36625" width="0.1524" layer="1"/>
+<wire x1="5.3975" y1="9.36625" x2="4.60375" y2="9.36625" width="0.1524" layer="1"/>
+<via x="4.28625" y="9.68375" extent="1-16" drill="0.2"/>
+<wire x1="4.28625" y1="9.68375" x2="4.28625" y2="10.4775" width="0.1524" layer="16"/>
+<wire x1="4.60375" y1="9.36625" x2="4.28625" y2="9.68375" width="0.1524" layer="1"/>
+<wire x1="6.0325" y1="10.00125" x2="6.066953125" y2="10.064721875" width="0" layer="19" extent="1-1"/>
+<wire x1="4.28625" y1="10.52125" x2="4.28625" y2="10.4775" width="0" layer="19" extent="16-16"/>
 <wire x1="6.0325" y1="10.16" x2="6.066953125" y2="10.064721875" width="0" layer="19" extent="1-1"/>
 </signal>
@@
 <wire x1="6.0325" y1="2.38125" x2="6.0325" y2="1.905" width="0.1524" layer="16"/>
 </signal>
-<signal name="C">
-<contactref element="LED1" pad="A"/>
-<contactref element="IC1" pad="19"/>
-<wire x1="7.14375" y1="8.89" x2="6.6675" y2="8.41375" width="0.1524" layer="1"/>
-<via x="4.445" y="9.525" extent="1-16" drill="0.2"/>
-<wire x1="6.6675" y1="8.41375" x2="5.55625" y2="8.41375" width="0.1524" layer="1"/>
-<wire x1="5.55625" y1="8.41375" x2="4.445" y2="9.525" width="0.1524" layer="1"/>
-<wire x1="4.445" y1="9.525" x2="4.28625" y2="9.68375" width="0.1524" layer="16"/>
-<wire x1="4.28625" y1="9.68375" x2="4.28625" y2="10.4775" width="0.1524" layer="16"/>
-<wire x1="4.28625" y1="10.4775" x2="4.28625" y2="10.52125" width="0" layer="19" extent="16-16"/>
-<wire x1="7.198325" y1="8.93335" x2="7.14375" y2="8.89" width="0" layer="19" extent="1-1"/>
-</signal>
 <signal name="N$36">
