File: Yaesu to CIV.brd (EAGLE design)
At the start: 24.9 x 20.9 mm, 56 parts, among them IC1 MEGA8-AI, IC2 MC78M05CDTG, Q1 16Mhz, Q2 BC857, Q3 BC857, Q4 BC849SMD

Commit message: Add files via upload
Parts:
- R12: value 4k7 -> 100k
- R7: value 4k7 -> 1k
Changed lines of the file:
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@@
 <attribute name="VALUE" x="22.225" y="2.2225" size="1.27" layer="27" rot="R90"/>
 </element>
-<element name="R12" library="rcl" library_urn="urn:adsk.eagle:library:334" package="R0603" package3d_urn="urn:adsk.eagle:package:23555/3" value="4k7" x="18.415" y="2.8575" smashed="yes" rot="R90">
+<element name="R12" library="rcl" library_urn="urn:adsk.eagle:library:334" package="R0603" package3d_urn="urn:adsk.eagle:package:23555/3" value="100k" x="18.415" y="2.8575" smashed="yes" rot="R90">
 <attribute name="NAME" x="19.20875" y="1.27" size="0.4064" layer="25" rot="R180"/>
 <attribute name="POPULARITY" value="70" x="66.675" y="30.7975" size="1.778" layer="27" rot="R90" display="off"/>
@@
 <attribute name="VALUE" x="6.6675" y="17.62125" size="1.27" layer="27" rot="R90"/>
 </element>
-<element name="R7" library="rcl" library_urn="urn:adsk.eagle:library:334" package="R0603" package3d_urn="urn:adsk.eagle:package:23555/3" value="4k7" x="16.03375" y="5.87375" smashed="yes" rot="R90">
+<element name="R7" library="rcl" library_urn="urn:adsk.eagle:library:334" package="R0603" package3d_urn="urn:adsk.eagle:package:23555/3" value="1k" x="16.03375" y="5.87375" smashed="yes" rot="R90">
 <attribute name="NAME" x="17.30375" y="5.87375" size="0.4064" layer="25" rot="R180"/>
 <attribute name="POPULARITY" value="70" x="69.37375" y="28.73375" size="1.778" layer="27" rot="R90" display="off"/>

Commit message: Add files via upload
Parts:
- added R10: 10k, rcl:R0603
- moved C5 0.45 mm to (10.9, 19.3)
- moved C1 0.45 mm to (11.9, 18.3)
- moved MOSI 0.32 mm to (8.10, 17.8)
Connections:
- removed net N$4: C3.1, C5.1, IC1.18, IC1.4, IC1.6, L1.2
- new net N$22: C3.1, C5.1, IC1.18, IC1.4, IC1.6, L1.2, R10.2
- net TX_IN: now also R10.1
Routing:
- net N$22: track 0.00 -> 35.6 mm, vias 0 -> 1
- net N$4: track 30.7 -> 0.00 mm, vias 1 -> 0
- net TX_IN: track 0.00 -> 8.04 mm
- net N$26: track 3.02 -> 0.00 mm
- net N$30: track 6.50 -> 6.00 mm
Other:
- board text added: "REV 3.2b"
