File: Yaesu to CIV.sch (EAGLE design)
At the start: 54 parts, among them IC1 MEGA8-AI, IC2 MC78M05CDTG, Q1 16Mhz, Q2 BC849SMD, Q3 BC849SMD, Q4 BC849SMD

Commit message: Add files via upload
Parts:
- added LED1: (no value), led:LEDCHIP-LED0603
- added R16: 470R7, rcl:R-EU_R0603
Connections:
- new net C: IC1.ADC6, LED1.A
- new net N$36: LED1.C, R16.1
- net GND: now also R16.2
Changed lines of the file:
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@@
 <part name="C14" library="rcl" library_urn="urn:adsk.eagle:library:334" deviceset="C-EU" device="C0603K" package3d_urn="urn:adsk.eagle:package:23680/2" value="100n"/>
 <part name="GND11" library="supply1" library_urn="urn:adsk.eagle:library:371" deviceset="GND" device=""/>
+<part name="LED1" library="led" deviceset="LED" device="CHIP-LED0603"/>
+<part name="R16" library="rcl" library_urn="urn:adsk.eagle:library:334" deviceset="R-EU_" device="R0603" package3d_urn="urn:adsk.eagle:package:23555/3" value="470R7"/>
+<part name="GND12" library="supply1" library_urn="urn:adsk.eagle:library:371" deviceset="GND" device=""/>
 </parts>
 <sheets>
@@
 <instance part="GND11" gate="1" x="190.5" y="62.23" smashed="yes">
 <attribute name="VALUE" x="187.96" y="59.69" size="1.778" layer="96"/>
+</instance>
+<instance part="LED1" gate="G$1" x="148.59" y="16.51" smashed="yes">
+<attribute name="NAME" x="152.146" y="11.938" size="1.778" layer="95" rot="R90"/>
+<attribute name="VALUE" x="154.305" y="11.938" size="1.778" layer="96" rot="R90"/>
+</instance>
+<instance part="R16" gate="G$1" x="148.59" y="5.08" smashed="yes" rot="R270">
+<attribute name="NAME" x="150.0886" y="8.89" size="1.778" layer="95" rot="R270"/>
+<attribute name="VALUE" x="145.288" y="8.89" size="1.778" layer="96" rot="R270"/>
+</instance>
+<instance part="GND12" gate="1" x="148.59" y="-2.54" smashed="yes">
+<attribute name="VALUE" x="146.05" y="-5.08" size="1.778" layer="96"/>
 </instance>
 </instances>
@@
 <pinref part="GND11" gate="1" pin="GND"/>
 </segment>
+<segment>
+<pinref part="R16" gate="G$1" pin="2"/>
+<pinref part="GND12" gate="1" pin="GND"/>
+</segment>
 </net>
 <net name="+5V" class="0">
@@
 </segment>
 </net>
+<net name="C" class="0">
+<segment>
+<wire x1="143.51" y1="30.48" x2="148.59" y2="30.48" width="0.1524" layer="91"/>
+<pinref part="LED1" gate="G$1" pin="A"/>
+<wire x1="148.59" y1="30.48" x2="148.59" y2="19.05" width="0.1524" layer="91"/>
+<pinref part="IC1" gate="G$1" pin="ADC6"/>
+<wire x1="124.46" y1="60.96" x2="143.51" y2="60.96" width="0.1524" layer="91"/>
+<wire x1="143.51" y1="60.96" x2="143.51" y2="30.48" width="0.1524" layer="91"/>
+</segment>
+</net>
+<net name="N$36" class="0">
+<segment>
+<pinref part="R16" gate="G$1" pin="1"/>
+<pinref part="LED1" gate="G$1" pin="C"/>
+<wire x1="148.59" y1="10.16" x2="148.59" y2="11.43" width="0.1524" layer="91"/>
+</segment>
+</net>

Commit message: Add files via upload
Connections:
- removed net C: IC1.ADC6, LED1.A
- net N$24: now also LED1.A
Changed lines of the file:
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@@
 <setting verticaltext="up"/>
 </settings>
-<grid distance="1.27" unitdist="mm" unit="mm" style="lines" multiple="1" display="no" altdistance="0.01" altunitdist="inch" altunit="inch"/>
+<grid distance="0.1" unitdist="inch" unit="inch" style="lines" multiple="1" display="no" altdistance="0.01" altunitdist="inch" altunit="inch"/>
 <layers>
 <layer number="1" name="Top" color="4" fill="1" visible="no" active="no"/>
@@
 <wire x1="124.46" y1="17.78" x2="125.73" y2="17.78" width="0.1524" layer="91"/>
 <pinref part="SCK" gate="1" pin="P"/>
+<wire x1="125.73" y1="17.78" x2="125.73" y2="15.24" width="0.1524" layer="91"/>
+<wire x1="125.73" y1="15.24" x2="142.24" y2="15.24" width="0.1524" layer="91"/>
+<junction x="125.73" y="17.78"/>
+<wire x1="142.24" y1="15.24" x2="142.24" y2="20.32" width="0.1524" layer="91"/>
+<pinref part="LED1" gate="G$1" pin="A"/>
+<wire x1="142.24" y1="20.32" x2="148.59" y2="20.32" width="0.1524" layer="91"/>
+<wire x1="148.59" y1="20.32" x2="148.59" y2="19.05" width="0.1524" layer="91"/>
 </segment>
 </net>
@@
 </segment>
 </net>
-<net name="C" class="0">
-<segment>
-<wire x1="143.51" y1="30.48" x2="148.59" y2="30.48" width="0.1524" layer="91"/>
-<pinref part="LED1" gate="G$1" pin="A"/>
-<wire x1="148.59" y1="30.48" x2="148.59" y2="19.05" width="0.1524" layer="91"/>
-<pinref part="IC1" gate="G$1" pin="ADC6"/>
-<wire x1="124.46" y1="60.96" x2="143.51" y2="60.96" width="0.1524" layer="91"/>
-<wire x1="143.51" y1="60.96" x2="143.51" y2="30.48" width="0.1524" layer="91"/>
-</segment>
-</net>
