File: Yaesu to CIV.sch (EAGLE design)
At the start: 56 parts, among them IC1 MEGA8-AI, IC2 MC78M05CDTG, Q1 16Mhz, Q2 BC857, Q3 BC857, Q4 BC849SMD

Commit message: Add files via upload
Parts:
- R12: value 4k7 -> 100k
- R7: value 4k7 -> 1k
Changed lines of the file:
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@@
 <part name="GND2" library="supply1" library_urn="urn:adsk.eagle:library:371" deviceset="GND" device=""/>
 <part name="R6" library="rcl" library_urn="urn:adsk.eagle:library:334" deviceset="R-EU_" device="R0603" package3d_urn="urn:adsk.eagle:package:23555/3" value="1k"/>
-<part name="R7" library="rcl" library_urn="urn:adsk.eagle:library:334" deviceset="R-EU_" device="R0603" package3d_urn="urn:adsk.eagle:package:23555/3" value="4k7"/>
+<part name="R7" library="rcl" library_urn="urn:adsk.eagle:library:334" deviceset="R-EU_" device="R0603" package3d_urn="urn:adsk.eagle:package:23555/3" value="1k"/>
 <part name="R11" library="rcl" library_urn="urn:adsk.eagle:library:334" deviceset="R-EU_" device="R0603" package3d_urn="urn:adsk.eagle:package:23555/3" value="10k"/>
 <part name="P+1" library="supply1" library_urn="urn:adsk.eagle:library:371" deviceset="+5V" device=""/>
 <part name="GND3" library="supply1" library_urn="urn:adsk.eagle:library:371" deviceset="GND" device=""/>
-<part name="R12" library="rcl" library_urn="urn:adsk.eagle:library:334" deviceset="R-EU_" device="R0603" package3d_urn="urn:adsk.eagle:package:23555/3" value="4k7"/>
+<part name="R12" library="rcl" library_urn="urn:adsk.eagle:library:334" deviceset="R-EU_" device="R0603" package3d_urn="urn:adsk.eagle:package:23555/3" value="100k"/>
 <part name="SCK" library="wirepad" library_urn="urn:adsk.eagle:library:412" deviceset="SMD2" device="" package3d_urn="urn:adsk.eagle:package:30839/1"/>
 <part name="MISO" library="wirepad" library_urn="urn:adsk.eagle:library:412" deviceset="SMD2" device="" package3d_urn="urn:adsk.eagle:package:30839/1"/>

Commit message: Add files via upload
Parts:
- added R10: 10k, rcl:R-EU_R0603
Connections:
- removed net N$4: C3.1, C5.1, IC1.AVCC, IC1.VCC@1, IC1.VCC@2, L1.2
- new net N$22: C3.1, C5.1, IC1.AVCC, IC1.VCC@1, IC1.VCC@2, L1.2, R10.2
- net TX_IN: now also R10.1
Changed lines of the file:
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@@
 <part name="L6" library="rcl" library_urn="urn:adsk.eagle:library:334" deviceset="L-EU" device="L2012C" package3d_urn="urn:adsk.eagle:package:23475/2"/>
 <part name="GND13" library="supply1" library_urn="urn:adsk.eagle:library:371" deviceset="GND" device=""/>
+<part name="R10" library="rcl" library_urn="urn:adsk.eagle:library:334" deviceset="R-EU_" device="R0603" package3d_urn="urn:adsk.eagle:package:23555/3" value="10k"/>
 </parts>
 <sheets>
@@
 <attribute name="VALUE" x="217.17" y="58.42" size="1.778" layer="96"/>
 </instance>
+<instance part="R10" gate="G$1" x="151.13" y="77.47" smashed="yes">
+<attribute name="NAME" x="147.32" y="78.9686" size="1.778" layer="95"/>
+<attribute name="VALUE" x="147.32" y="74.168" size="1.778" layer="96"/>
+</instance>
 </instances>
 <busses>
@@
 <wire x1="50.8" y1="52.07" x2="50.8" y2="53.34" width="0.1524" layer="91"/>
 <junction x="50.8" y="53.34"/>
-</segment>
-</net>
-<net name="N$4" class="0">
-<segment>
-<pinref part="IC1" gate="G$1" pin="VCC@2"/>
-<wire x1="76.2" y1="38.1" x2="73.66" y2="38.1" width="0.1524" layer="91"/>
-<wire x1="73.66" y1="38.1" x2="73.66" y2="40.64" width="0.1524" layer="91"/>
-<pinref part="IC1" gate="G$1" pin="VCC@1"/>
-<wire x1="73.66" y1="40.64" x2="76.2" y2="40.64" width="0.1524" layer="91"/>
-<wire x1="73.66" y1="38.1" x2="67.31" y2="38.1" width="0.1524" layer="91"/>
-<junction x="73.66" y="38.1"/>
-<pinref part="C3" gate="G$1" pin="1"/>
-<wire x1="67.31" y1="38.1" x2="59.69" y2="38.1" width="0.1524" layer="91"/>
-<wire x1="73.66" y1="35.56" x2="73.66" y2="38.1" width="0.1524" layer="91"/>
-<pinref part="L1" gate="G$1" pin="2"/>
-<pinref part="IC1" gate="G$1" pin="AVCC"/>
-<wire x1="76.2" y1="66.04" x2="67.31" y2="66.04" width="0.1524" layer="91"/>
-<wire x1="67.31" y1="66.04" x2="67.31" y2="38.1" width="0.1524" layer="91"/>
-<junction x="67.31" y="38.1"/>
-<pinref part="C5" gate="G$1" pin="1"/>
-<wire x1="67.31" y1="66.04" x2="38.1" y2="66.04" width="0.1524" layer="91"/>
-<wire x1="38.1" y1="66.04" x2="38.1" y2="52.07" width="0.1524" layer="91"/>
-<junction x="67.31" y="66.04"/>
 </segment>
 </net>
@@
 <segment>
 <wire x1="153.67" y1="102.87" x2="144.78" y2="102.87" width="0.1524" layer="91"/>
-<wire x1="144.78" y1="102.87" x2="144.78" y2="66.04" width="0.1524" layer="91"/>
+<wire x1="144.78" y1="102.87" x2="144.78" y2="77.47" width="0.1524" layer="91"/>
 <pinref part="R6" gate="G$1" pin="1"/>
+<wire x1="144.78" y1="77.47" x2="144.78" y2="66.04" width="0.1524" layer="91"/>
 <wire x1="144.78" y1="66.04" x2="138.43" y2="66.04" width="0.1524" layer="91"/>
 <pinref part="X1" gate="-1" pin="7"/>
 <wire x1="153.67" y1="100.33" x2="153.67" y2="102.87" width="0.1524" layer="91"/>
+<pinref part="R10" gate="G$1" pin="1"/>
+<wire x1="146.05" y1="77.47" x2="144.78" y2="77.47" width="0.1524" layer="91"/>
+<junction x="144.78" y="77.47"/>
 </segment>
 </net>
@@
 </segment>
 </net>
+<net name="N$22" class="0">
+<segment>
+<pinref part="R10" gate="G$1" pin="2"/>
+<wire x1="156.21" y1="77.47" x2="157.48" y2="77.47" width="0.1524" layer="91"/>
+<label x="157.48" y="77.47" size="1.778" layer="95" xref="yes"/>
+</segment>
+<segment>
+<pinref part="IC1" gate="G$1" pin="VCC@2"/>
+<wire x1="76.2" y1="38.1" x2="73.66" y2="38.1" width="0.1524" layer="91"/>
+<wire x1="73.66" y1="38.1" x2="73.66" y2="40.64" width="0.1524" layer="91"/>
+<pinref part="IC1" gate="G$1" pin="VCC@1"/>
+<wire x1="73.66" y1="40.64" x2="76.2" y2="40.64" width="0.1524" layer="91"/>
+<wire x1="73.66" y1="38.1" x2="67.31" y2="38.1" width="0.1524" layer="91"/>
+<junction x="73.66" y="38.1"/>
+<pinref part="C3" gate="G$1" pin="1"/>
+<wire x1="67.31" y1="38.1" x2="59.69" y2="38.1" width="0.1524" layer="91"/>
+<wire x1="73.66" y1="35.56" x2="73.66" y2="38.1" width="0.1524" layer="91"/>
+<pinref part="L1" gate="G$1" pin="2"/>
+<pinref part="IC1" gate="G$1" pin="AVCC"/>
+<wire x1="76.2" y1="66.04" x2="67.31" y2="66.04" width="0.1524" layer="91"/>
+<wire x1="67.31" y1="66.04" x2="67.31" y2="38.1" width="0.1524" layer="91"/>
+<junction x="67.31" y="38.1"/>
+<pinref part="C5" gate="G$1" pin="1"/>
+<wire x1="67.31" y1="66.04" x2="38.1" y2="66.04" width="0.1524" layer="91"/>
+<wire x1="38.1" y1="66.04" x2="38.1" y2="52.07" width="0.1524" layer="91"/>
+<junction x="67.31" y="66.04"/>
+<wire x1="67.31" y1="38.1" x2="67.31" y2="36.83" width="0.1524" layer="91"/>
+<label x="67.31" y="36.83" size="1.778" layer="95" rot="R270" xref="yes"/>
+</segment>
+</net>
